Commit message: Added Camera to the arm

File: src/ur5e_zivid_config/config/gazebo_ur5e_zivid.urdf (robot description, URDF)
Before this commit: robot ur5e_zivid, 17 links, 16 joints
Links:
- added link camera_link
Joints:
- added joint camera_joint: type fixed, parent zivid_optical_center, child camera_link, origin xyz=0.0 0.0 0.05 rpy=1.570795 -1.570795 0
